File: breakout.kicad_pcb (KiCad board)
At the start: 2 copper layers, 50 x 50 mm, 100 parts

Commit message: gerber.
Parts:
- added REF**: R_0805, Resistors_SMD:R_0805, B.Cu at (130.8, 111.3)
- added REF**: R_0805, Resistors_SMD:R_0805, B.Cu at (130.8, 117.5)
- added REF**: R_0805, Resistors_SMD:R_0805, B.Cu at (143.5, 117.5)
- added REF**: R_0805, Resistors_SMD:R_0805, B.Cu at (143.5, 111.3)
- added REF**: R_0805, Resistors_SMD:R_0805, B.Cu at (143.5, 101.1)
- added REF**: R_0805, Resistors_SMD:R_0805, B.Cu at (143.5, 107.3)
- added REF**: R_0805, Resistors_SMD:R_0805, B.Cu at (130.8, 107.3)
- added REF**: R_0805, Resistors_SMD:R_0805, B.Cu at (130.8, 101.1)
- added REF**: R_0805, Resistors_SMD:R_0805, B.Cu at (118.1, 101.1)
- added REF**: R_0805, Resistors_SMD:R_0805, B.Cu at (118.1, 107.3)
- added REF**: R_0805, Resistors_SMD:R_0805, B.Cu at (105.4, 107.3)
- added REF**: R_0805, Resistors_SMD:R_0805, B.Cu at (105.4, 101.1)
- added REF**: R_0805, Resistors_SMD:R_0805, B.Cu at (130.8, 141.7)
- added REF**: R_0805, Resistors_SMD:R_0805, B.Cu at (130.8, 148.0)
- added REF**: R_0805, Resistors_SMD:R_0805, B.Cu at (143.5, 148.0)
- added REF**: R_0805, Resistors_SMD:R_0805, B.Cu at (143.5, 141.7)
- added REF**: R_0805, Resistors_SMD:R_0805, B.Cu at (105.4, 121.4)
- added REF**: R_0805, Resistors_SMD:R_0805, B.Cu at (105.4, 127.6)
- added REF**: R_0805, Resistors_SMD:R_0805, B.Cu at (118.1, 127.6)
- added REF**: R_0805, Resistors_SMD:R_0805, B.Cu at (118.1, 121.4)
- added REF**: R_0805, Resistors_SMD:R_0805, B.Cu at (130.8, 121.4)
- added REF**: R_0805, Resistors_SMD:R_0805, B.Cu at (130.8, 127.6)
- added REF**: R_0805, Resistors_SMD:R_0805, B.Cu at (143.5, 127.6)
- added REF**: R_0805, Resistors_SMD:R_0805, B.Cu at (143.5, 121.4)
- added REF**: R_0805, Resistors_SMD:R_0805, B.Cu at (105.4, 141.7)
- added REF**: R_0805, Resistors_SMD:R_0805, B.Cu at (143.5, 131.6)
- added REF**: R_0805, Resistors_SMD:R_0805, B.Cu at (143.5, 137.8)
- added REF**: R_0805, Resistors_SMD:R_0805, B.Cu at (130.8, 137.8)
- added REF**: R_0805, Resistors_SMD:R_0805, B.Cu at (130.8, 131.6)
- added REF**: R_0805, Resistors_SMD:R_0805, B.Cu at (105.4, 148.0)
- added REF**: R_0805, Resistors_SMD:R_0805, B.Cu at (118.1, 131.6)
- added REF**: R_0805, Resistors_SMD:R_0805, B.Cu at (118.1, 137.8)
- added REF**: R_0805, Resistors_SMD:R_0805, B.Cu at (105.4, 137.8)
- added REF**: R_0805, Resistors_SMD:R_0805, B.Cu at (105.4, 131.6)
- added REF**: R_0805, Resistors_SMD:R_0805, B.Cu at (118.1, 148.0)
- added REF**: R_0805, Resistors_SMD:R_0805, B.Cu at (118.1, 141.7)
- added REF**: R_0805, Resistors_SMD:R_0805, B.Cu at (105.4, 111.3)
- added REF**: R_0805, Resistors_SMD:R_0805, B.Cu at (105.4, 117.5)
- added REF**: R_0805, Resistors_SMD:R_0805, B.Cu at (118.1, 117.5)
- added REF**: R_0805, Resistors_SMD:R_0805, B.Cu at (118.1, 111.3)
Routing:
- net (no net): track 896.9 -> 1277.7 mm
Other:
- board text removed: "SOT-23"
- board text removed: "SOT-23-6"
